File: breast-module-proto-v1/kicad/psu.kicad_sch (KiCad schematic)
At the start: 41 parts, among them SW1 power on, SW2 power off, U1 AMS1117-3.3, U2 TP4056, U3 TPS61230ARNSR, U4 DW01, U5 FS8205A, U6 74HC00

Commit message: Changed battery connector footprint
Parts:
- BT1: footprint Connector_JST:JST_XH_S2B-XH-A-1_1x02_P2.50mm_Horizontal -> Connector_JST:JST_XH_S2B-XH-A_1x02_P2.50mm_Horizontal
Changed lines of the file:
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@@
       (effects (font (size 1.27 1.27)) (justify left))
     )
-    (property "Footprint" "Connector_JST:JST_XH_S2B-XH-A-1_1x02_P2.50mm_Horizontal" (id 2) (at 151.13 166.116 90)
+    (property "Footprint" "Connector_JST:JST_XH_S2B-XH-A_1x02_P2.50mm_Horizontal" (id 2) (at 151.13 166.116 90)
       (effects (font (size 1.27 1.27)) hide)
     )
