File: chest-module-proto-v1/kicad/chest-module-proto-v1.kicad_sch (KiCad schematic)
At the start: 0 parts

Commit message: Renamed strings
Other:
- title: Breast Module -> Chest Module
Changed lines of the file:
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@@
   (paper "A4")
   (title_block
-    (title "Breast Module")
+    (title "Chest Module")
     (date "2023-01-28")
     (rev "Proto V1")
