File: chest-module-proto-v1/kicad/cpu.kicad_sch (KiCad schematic)
At the start: 23 parts, among them J1 USB_C_Receptacle_USB2.0, J2 Conn_01x06_Male, J3 Conn_01x06_Male, Q1 SS8050-G, Q2 SS8050-G, U7 ESP32-WROOM-32, U8 USBLC6-2SC6, U9 CP2102N-Axx-xQFN28

Commit message: Renamed strings
Other:
- title: Breast Module -> Chest Module
Changed lines of the file:
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@@
   (paper "A4")
   (title_block
-    (title "Breast Module")
+    (title "Chest Module")
     (date "2023-01-28")
     (rev "Proto V1")
