File: chest-module-proto-v1/kicad/hitpoint.kicad_sch (KiCad schematic)
At the start: 32 parts, among them J4 SWD, U10 74HC00, U11 IRM-H6XXT, U12 IRM-H6XXT, U13 STM32G030Fx

Commit message: Renamed strings
Other:
- note added: "MCFG Table: 000: Phaser 001: Chest 010: Back 011: Shoulder L 100: Shoulder R 101: Head 110: Hitpoint 111: -"
- note removed: "MCFG Table: 000: Phaser 001: Breast 010: Back 011: Shoulder L 100: Shoulder R 101: Head 110: Hitpoint 111: -"
- title: Breast Module -> Chest Module
Changed lines of the file:
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@@
   (paper "A4")
   (title_block
-    (title "Breast Module")
+    (title "Chest Module")
     (date "2023-01-28")
     (rev "Proto V1")
@@
     (stroke (width 0) (type default) (color 0 0 0 0))
   )
-  (text "MCFG Table:\n\n000: Phaser\n001: Breast\n010: Back\n011: Shoulder L\n100: Shoulder R\n101: Head\n110: Hitpoint\n111: -"
+  (text "MCFG Table:\n\n000: Phaser\n001: Chest\n010: Back\n011: Shoulder L\n100: Shoulder R\n101: Head\n110: Hitpoint\n111: -"
     (at 241.3 127 0)
     (effects (font (size 1.27 1.27)) (justify left bottom))
