File: chest-module-proto-v1/kicad/psu.kicad_sch (KiCad schematic)
At the start: 41 parts, among them SW1 power on, SW2 power off, U1 AMS1117-3.3, U2 TP4056, U3 TPS61230ARNSR, U4 DW01, U5 FS8205A, U6 74HC00

Commit message: Renamed strings
Other:
- title: Breast Module -> Chest Module
Changed lines of the file:
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@@
   (paper "A4")
   (title_block
-    (title "Breast Module")
+    (title "Chest Module")
     (date "2023-01-28")
     (rev "Proto V1")
